File: V2/PCB/McPiFace-Status-V2.brd (EAGLE design)
At the start: 88 x 88 mm, 36 parts, among them IC1 MCP23017SO, J1 MC_PI_FACE_CONNECTORS_LEDSSIDE

Commit message: Updated LEDs used to use the larger hole version.
Parts:
- D2, D3: device ThingySticks:LED-1206-BOTTOM-1.6MM -> ThingySticks:LED-1206-BOTTOM-2.0MM
- moved R1 0.10 mm to (10.0, 53.4)
Other:
- board text added: "McPiFace.com"
- board text removed: "MyPiFace.com"
- board text removed: "PiBlade McStatus PiFace"
Changed lines of the file:
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@@
 <grid distance="0.1" unitdist="mm" unit="mm" style="lines" multiple="1" display="yes" altdistance="0.1" altunitdist="mm" altunit="mm"/>
 <layers>
-<layer number="1" name="Top" color="4" fill="1" visible="no" active="yes"/>
+<layer number="1" name="Top" color="4" fill="1" visible="yes" active="yes"/>
 <layer number="2" name="Route2" color="1" fill="3" visible="no" active="no"/>
 <layer number="3" name="Route3" color="4" fill="3" visible="no" active="no"/>
@@
 <layer number="19" name="Unrouted" color="6" fill="1" visible="yes" active="yes"/>
 <layer number="20" name="Dimension" color="15" fill="1" visible="yes" active="yes"/>
-<layer number="21" name="tPlace" color="7" fill="1" visible="no" active="yes"/>
+<layer number="21" name="tPlace" color="7" fill="1" visible="yes" active="yes"/>
 <layer number="22" name="bPlace" color="7" fill="1" visible="yes" active="yes"/>
 <layer number="23" name="tOrigins" color="15" fill="1" visible="yes" active="yes"/>
 <layer number="24" name="bOrigins" color="15" fill="1" visible="yes" active="yes"/>
-<layer number="25" name="tNames" color="7" fill="1" visible="no" active="yes"/>
+<layer number="25" name="tNames" color="7" fill="1" visible="yes" active="yes"/>
 <layer number="26" name="bNames" color="7" fill="1" visible="yes" active="yes"/>
 <layer number="27" name="tValues" color="7" fill="1" visible="yes" active="yes"/>
@@
 <wire x1="-1.5" y1="76" x2="100" y2="76" width="0.4064" layer="49"/>
 <wire x1="-3.5" y1="12" x2="100" y2="12" width="0.4064" layer="49"/>
-<text x="43.1" y="15.1" size="1.778" layer="1" ratio="15">PiBlade McStatus PiFace</text>
 <text x="86.3225" y="17.5925" size="1.778" layer="26" ratio="15" rot="MR0">http://github.com/McPiFace/Status</text>
 <circle x="22" y="82" radius="5" width="0" layer="41"/>
@@
 <text x="86.0225" y="11.9925" size="1.778" layer="26" ratio="15" rot="MR0">S.Harrison
 9 Feb 2019</text>
-<text x="56.6225" y="80.8925" size="2.54" layer="26" ratio="15" rot="MR0">MyPiFace.com</text>
+<text x="56.6225" y="80.8925" size="2.54" layer="26" ratio="15" rot="MR0">McPiFace.com</text>
 <text x="73.69" y="28.9" size="1.27" layer="26" ratio="15" rot="MR0">3v3</text>
 <text x="44" y="64.5" size="1.016" layer="26" ratio="15" rot="MR0">GPA7</text>
@@
 </class>
 </classes>
-<designrules name="dirt_cheap_dirty_boards.v1">
+<designrules name="dirt_cheap_dirty_boards.v1.1">
+<description language="de">&lt;b&gt;Dirty Cheap Dirty Board Design Rules&lt;/b&gt;
+&lt;br&gt;
+&lt;br&gt;Min width/Spacing: 6/6mil
+&lt;br&gt;Min diameter of finished hole 12mil</description>
 <description language="en">&lt;b&gt;Dirty Cheap Dirty Board Design Rules&lt;/b&gt;
 &lt;br&gt;
-&lt;br&gt;Min width/Spacing: 5/5mil
+&lt;br&gt;Min width/Spacing: 6/6mil
+&lt;br&gt;Min diameter of finished hole 12mil</description>
+<description language="zh">&lt;b&gt;Dirty Cheap Dirty Board Design Rules&lt;/b&gt;
+&lt;br&gt;
+&lt;br&gt;Min width/Spacing: 6/6mil
 &lt;br&gt;Min diameter of finished hole 12mil</description>
 <param name="layerSetup" value="(1*16)"/>
 <param name="mtCopper" value="0.035mm 0.0175mm 0.035mm 0.035mm 0.035mm 0.035mm 0.035mm 0.035mm 0.035mm 0.035mm 0.035mm 0.035mm 0.035mm 0.035mm 0.0175mm 0.035mm"/>
 <param name="mtIsolate" value="1.5mm 1.1mm 0.2mm 0.15mm 0.2mm 0.15mm 0.2mm 0.15mm 0.2mm 0.15mm 0.2mm 0.15mm 0.2mm 0.15mm 0.2mm"/>
-<param name="mdWireWire" value="5mil"/>
-<param name="mdWirePad" value="5mil"/>
-<param name="mdWireVia" value="5mil"/>
-<param name="mdPadPad" value="5mil"/>
-<param name="mdPadVia" value="5mil"/>
-<param name="mdViaVia" value="5mil"/>
+<param name="mdWireWire" value="6mil"/>
+<param name="mdWirePad" value="6mil"/>
+<param name="mdWireVia" value="6mil"/>
+<param name="mdPadPad" value="6mil"/>
+<param name="mdPadVia" value="6mil"/>
+<param name="mdViaVia" value="6mil"/>
 <param name="mdSmdPad" value="0mil"/>
 <param name="mdSmdVia" value="0mil"/>
@@
 <param name="mdDrill" value="10mil"/>
 <param name="mdSmdStop" value="0mil"/>
-<param name="msWidth" value="5mil"/>
+<param name="msWidth" value="6mil"/>
 <param name="msDrill" value="12mil"/>
 <param name="msMicroVia" value="12mil"/>
@@
 <elements>
 <element name="LOGO1" library="SparkFun-Aesthetics" package="OSHW-LOGO-L" value="OSHW-LOGOL" x="44" y="6" rot="MR0"/>
-<element name="D2" library="ThingySticks" package="LED-1206-BOTTOM-1.6MM" value="" x="4" y="59" smashed="yes" rot="MR90">
+<element name="D2" library="ThingySticks" package="LED-1206-BOTTOM-2.0MM" value="" x="4" y="59" smashed="yes" rot="MR90">
 <attribute name="VALUE" x="2.73" y="59" size="0.6096" layer="28" font="vector" ratio="20" rot="MR90" align="top-center"/>
-</element>
-<element name="D3" library="ThingySticks" package="LED-1206-BOTTOM-1.6MM" value="" x="10" y="59" smashed="yes" rot="MR90">
+<attribute name="COLOR" value="Green" x="4" y="59" size="1.778" layer="28" rot="MR90" display="off"/>
+<attribute name="FARNELL" value="2217905" x="4" y="59" size="1.778" layer="28" rot="MR90" display="off"/>
+<attribute name="FORWARD_VOLTAGE" value="2.1" x="4" y="59" size="1.778" layer="28" rot="MR90" display="off"/>
+</element>
+<element name="D3" library="ThingySticks" package="LED-1206-BOTTOM-2.0MM" value="" x="10" y="59" smashed="yes" rot="MR90">
 <attribute name="VALUE" x="8.73" y="59" size="0.6096" layer="28" font="vector" ratio="20" rot="MR90" align="top-center"/>
-</element>
-<element name="R1" library="SparkFun-Resistors" package="0805" value=" " x="10" y="53.3" smashed="yes" rot="MR90">
-<attribute name="PROD_ID" value=" " x="10" y="53.3" size="1.778" layer="28" rot="MR90" display="off"/>
+<attribute name="COLOR" value="Hyper Red" x="10" y="59" size="1.778" layer="28" rot="MR90" display="off"/>
+<attribute name="FARNELL" value="2217903" x="10" y="59" size="1.778" layer="28" rot="MR90" display="off"/>
+<attribute name="FORWARD_VOLTAGE" value="1.95" x="10" y="59" size="1.778" layer="28" rot="MR90" display="off"/>
+</element>
+<element name="R1" library="SparkFun-Resistors" package="0805" value=" " x="10" y="53.4" smashed="yes" rot="MR90">
+<attribute name="PROD_ID" value=" " x="10" y="53.4" size="1.778" layer="28" rot="MR90" display="off"/>
 </element>
 <element name="R2" library="SparkFun-Resistors" package="0805" value=" " x="4" y="53.4" smashed="yes" rot="MR90">
@@
 <attribute name="MFG" value="SM04B-SRSS-TB(LF)(SN)" x="6.8" y="49.8" size="1.778" layer="28" rot="MR0" display="off"/>
 <attribute name="FARNELL" value="1830839" x="6.8" y="49.8" size="1.778" layer="28" rot="MR0" display="off"/>
-<attribute name="NAME" x="7.197" y="46.341" size="0.6096" layer="26" font="vector" ratio="20" rot="MR0"/>
 </element>
 <element name="D4" library="ThingySticks" package="LED-1206-BOTTOM-2.0MM" value="GREEN" x="37.5" y="65" smashed="yes" rot="MR0">
@@
 <contactref element="D3" pad="A"/>
 <contactref element="R1" pad="2"/>
-<wire x1="10" y1="54.2" x2="10" y2="57.2" width="0.3048" layer="16"/>
+<wire x1="10" y1="54.3" x2="10" y2="57.2" width="0.3048" layer="16"/>
 </signal>
 <signal name="N$5">
@@
 <wire x1="7.3" y1="52" x2="7.6" y2="52.3" width="0.3048" layer="16"/>
 <wire x1="7.6" y1="52.3" x2="9.6" y2="52.3" width="0.3048" layer="16"/>
-<wire x1="9.6" y1="52.3" x2="10" y2="52.4" width="0.3048" layer="16"/>
+<wire x1="9.6" y1="52.3" x2="10" y2="52.5" width="0.3048" layer="16"/>
 </signal>
 <signal name="N$6">
