File: V2/PCB/McPiFace-Status-V2.sch (EAGLE design)
At the start: 36 parts, among them IC1 MCP23017SO, J1 MC_PI_FACE_CONNECTORS_LEDSSIDE

Commit message: Updated LEDs used to use the larger hole version.
Parts:
- D2: device ThingySticks:LED1206-BOTTOM-1.6MM -> ThingySticks:LEDLED-1206-BOTTOM-2.0MM-GREEN
- D3: device ThingySticks:LED1206-BOTTOM-1.6MM -> ThingySticks:LEDLED-1206-BOTTOM-2.0MM-RED
Changed lines of the file:
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@@
 <parts>
 <part name="LOGO1" library="SparkFun-Aesthetics" deviceset="OSHW-LOGO" device="L"/>
-<part name="D2" library="ThingySticks" deviceset="LED" device="1206-BOTTOM-1.6MM"/>
-<part name="D3" library="ThingySticks" deviceset="LED" device="1206-BOTTOM-1.6MM"/>
+<part name="D2" library="ThingySticks" deviceset="LED" device="LED-1206-BOTTOM-2.0MM-GREEN"/>
+<part name="D3" library="ThingySticks" deviceset="LED" device="LED-1206-BOTTOM-2.0MM-RED"/>
 <part name="R1" library="SparkFun-Resistors" deviceset="RESISTOR" device="0805" value=" "/>
 <part name="R2" library="SparkFun-Resistors" deviceset="RESISTOR" device="0805" value=" "/>
